File: kicad/pyp/pyp.kicad_pcb (KiCad board)
At the start: 2 copper layers, 14 x 24 mm, 11 parts, among them J1 Conn_01x04, SW1 SW_DIP_x01, U1 MSP430G2001IPW14

Commit message: v1.0
Parts:
- moved C2 1.44 mm to (177.8, -11.4)
- moved J1 1.44 mm to (172.2, -14.0)
- moved R1 1.37 mm to (177.8, -9.65)
- moved C1 1.33 mm to (177.8, -7.87)
- moved C3 1.33 mm to (177.8, -6.10)
- moved U1 0.53 mm to (179.1, -0.89)
- moved SW1 0.06 mm to (170.9, -6.75)
- renumbered Batt1 to Bat1
Routing:
- net GND: track 5.42 -> 18.2 mm, vias 1 -> 0
- net SBWTDIO: track 28.3 -> 20.7 mm, vias 1 -> 0
- net SBWTCK: track 17.4 -> 10.5 mm, vias 1 -> 0
- net VCC: track 28.4 -> 24.6 mm
- net Net-(U1-Pad13): track 0.00 -> 0.74 mm
- net Net-(Btn1-Pad1): track 8.45 -> 9.15 mm
Other:
- board text added: "3.3V"
- board text added: "CLK"
- board text added: "DIO"
- board text added: "GND"
