File: kicad/pyp/pyp.sch (KiCad schematic (older format))
At the start: 11 parts, among them J1 Conn_01x04, SW1 SW_DIP_x01, U1 MSP430G2001IPW14

Commit message: v1.0
Parts:
- renumbered Batt1 to Bat1
Changed lines of the file:
@@
 $EndComp
 $Comp
-L Device:Battery Batt1
+L Device:Battery Bat1
 U 1 1 5EC6DDF5
 P 6600 5200
-F 0 "Batt1" H 6708 5246 50  0000 L CNN
+F 0 "Bat1" H 6708 5246 50  0000 L CNN
 F 1 "3V" H 6708 5155 50  0000 L CNN
 F 2 "Connector_Wire:SolderWire-0.1sqmm_1x02_P3.6mm_D0.4mm_OD1mm" V 6600 5260 50  0001 C CNN
